File: rio hub/rio hub.kicad_pcb (KiCad board)
At the start: 2 copper layers, 160.8 x 155.2 mm, 1 part

Commit message: fixed diode placement, major rio hub work
Parts:
- added D1: D_Schottky, Diode_THT:D_DO-41_SOD81_P10.16mm_Horizontal, F.Cu at (135.2, 72.8)
- added J1: Conn_01x02_Pin, Connector_PinHeader_2.54mm:PinHeader_1x02_P2.54mm_Vertical, F.Cu at (106.5, 87.0)
- added J2: Conn_01x02_Pin, TerminalBlock_WAGO:TerminalBlock_WAGO_2601-1102_1x02_P3.50mm_Horizontal, F.Cu at (110.5, 78.4)
- added J3: Conn_01x02_Pin, Connector_PinHeader_2.54mm:PinHeader_1x02_P2.54mm_Vertical, F.Cu at (106.5, 71.0)
- added J4: MTJ-88ARX1-FSM-LG, custom:ADAMTECH_MTJ-88ARX1-FSM-LG, F.Cu at (149.2, 83.5)
- added J5: Conn_02x17_Odd_Even, Connector_PinSocket_2.54mm:PinSocket_2x17_P2.54mm_Vertical, F.Cu at (150.3, 127.3)
- added J6: Conn_01x04_Socket, Connector_PinSocket_2.54mm:PinSocket_1x04_P2.54mm_Vertical, F.Cu at (126.4, 114.0)
- added R1: R, Resistor_THT:R_Axial_DIN0207_L6.3mm_D2.5mm_P10.16mm_Horizontal, F.Cu at (135.1, 76.5)
- U1: footprint FRC:RoboRIO-THT -> FRC:RoboRIO_MXP-THT
- moved U1 7.49 mm to (105.2, 63.9)
Connections:
- U1 pad 1: unconnected-(U1I-MXP_5V-Pad1) -> Net-(J5-Pin_1)
- U1 pad 10: unconnected-(U1I-MXP_RX-Pad10) -> Net-(J5-Pin_10)
- U1 pad 11: unconnected-(U1I-MXP_DIO0_PWM0-Pad11) -> Net-(J5-Pin_11)
- U1 pad 12: unconnected-(U1I-MXP_DGND-Pad12) -> /DGND
- U1 pad 13: unconnected-(U1I-MXP_DIO1_PWM1-Pad13) -> Net-(J5-Pin_13)
- U1 pad 14: unconnected-(U1I-MXP_TX-Pad14) -> Net-(J5-Pin_14)
- U1 pad 15: unconnected-(U1I-MXP_DIO2_PWM2-Pad15) -> Net-(J5-Pin_15)
- U1 pad 16: unconnected-(U1I-MXP_DGND-Pad16) -> /DGND
- U1 pad 17: unconnected-(U1I-MXP_DIO3_PWM3-Pad17) -> Net-(J5-Pin_17)
- U1 pad 18: unconnected-(U1I-MXP_DIO11_PWM7-Pad18) -> Net-(J5-Pin_18)
- U1 pad 19: unconnected-(U1I-MXP_DIO4_CS-Pad19) -> Net-(J5-Pin_19)
- U1 pad 2: unconnected-(U1I-MXP_AO0-Pad2) -> Net-(J5-Pin_2)
- U1 pad 20: unconnected-(U1I-MXP_DGND-Pad20) -> /DGND
- U1 pad 21: unconnected-(U1I-MXP_DIO5_SCLK-Pad21) -> Net-(J5-Pin_21)
- U1 pad 22: unconnected-(U1I-MXP_DIO12_PWM8-Pad22) -> Net-(J5-Pin_22)
- U1 pad 23: unconnected-(U1I-MXP_DIO6_MISO-Pad23) -> Net-(J5-Pin_23)
- U1 pad 24: unconnected-(U1I-MXP_DGND-Pad24) -> /DGND
- U1 pad 25: unconnected-(U1I-MXP_DIO7_MOSI-Pad25) -> Net-(J5-Pin_25)
- U1 pad 26: unconnected-(U1I-MXP_DIO13_PWM9-Pad26) -> Net-(J5-Pin_26)
- U1 pad 27: unconnected-(U1I-MXP_DIO8_PWM4-Pad27) -> Net-(J5-Pin_27)
- U1 pad 28: unconnected-(U1I-MXP_DGND-Pad28) -> /DGND
- U1 pad 29: unconnected-(U1I-MXP_DIO9_PWM5-Pad29) -> Net-(J5-Pin_29)
- U1 pad 3: unconnected-(U1I-MXP_AI0-Pad3) -> Net-(J5-Pin_3)
- U1 pad 30: unconnected-(U1I-MXP_DGND-Pad30) -> /DGND
- U1 pad 31: unconnected-(U1I-MXP_DIO10_PWM6-Pad31) -> Net-(J5-Pin_31)
- U1 pad 32: unconnected-(U1I-MXP_DIO14_SCL-Pad32) -> Net-(J5-Pin_32)
- U1 pad 33: unconnected-(U1I-MXP_3V3-Pad33) -> Net-(J5-Pin_33)
- U1 pad 34: unconnected-(U1I-MXP_DIO15_SDA-Pad34) -> Net-(J5-Pin_34)
- U1 pad 4: unconnected-(U1I-MXP_AO1-Pad4) -> Net-(J5-Pin_4)
- U1 pad 5: unconnected-(U1I-MXP_AI1-Pad5) -> Net-(J5-Pin_5)
- U1 pad 6: unconnected-(U1I-MXP_AGND-Pad6) -> /AGND
- U1 pad 7: unconnected-(U1I-MXP_AI2-Pad7) -> Net-(J5-Pin_7)
- U1 pad 8: unconnected-(U1I-MXP_DGND-Pad8) -> /DGND
- U1 pad 9: unconnected-(U1I-MXP_AI3-Pad9) -> Net-(J5-Pin_9)
Routing:
- net /DGND: track 0.00 -> 95.9 mm
- net /12v: track 0.00 -> 52.4 mm
- net Net-(J1-Pin_1): track 0.00 -> 43.1 mm
- net Net-(J1-Pin_2): track 0.00 -> 42.0 mm
- net Net-(J6-Pin_1): track 0.00 -> 39.7 mm
- net Net-(J6-Pin_2): track 0.00 -> 35.6 mm
- net Net-(J6-Pin_3): track 0.00 -> 35.5 mm
- net Net-(J6-Pin_4): track 0.00 -> 31.4 mm
- net Net-(D1-A): track 0.00 -> 16.9 mm
- net Net-(J5-Pin_27): track 0.00 -> 9.09 mm
- net Net-(J5-Pin_4): track 0.00 -> 8.89 mm
- net Net-(J5-Pin_18): track 0.00 -> 8.89 mm
- net Net-(J5-Pin_10): track 0.00 -> 8.89 mm
- net Net-(J5-Pin_7): track 0.00 -> 8.89 mm
- net Net-(J5-Pin_34): track 0.00 -> 8.89 mm
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- added copper zone on B.Cu, net /DGND
- added copper zone on F.Cu, net /DGND
- added copper zone on B.Cu, net /GND
- added copper zone on F.Cu, net /GND
Other:
- board size 160.8 x 155.2 mm -> 58.2 x 80.5 mm

Commit message: rio hub work
Parts:
- moved D1 56.4 mm to (133.4, 129.1)
- moved J2 51.4 mm to (107.6, 129.8)
- moved J3 49.9 mm to (104.3, 120.8)
- moved J4 48.1 mm to (151.3, 131.6)
- moved R1 48.1 mm to (133.4, 124.6)
- moved J6 47.0 mm to (125.7, 161.0)
- moved U1 39.6 mm to (103.5, 103.5)
- moved J5 39.6 mm to (148.6, 166.9)
- moved J1 27.4 mm to (104.3, 114.3)
Routing:
- net /12v: track 52.4 -> 62.9 mm
- net Net-(J1-Pin_2): track 42.0 -> 49.0 mm
- net Net-(J1-Pin_1): track 43.1 -> 50.1 mm
- net Net-(J4-Pad9): track 5.09 -> 8.84 mm
- net Net-(J6-Pin_2): track 35.6 -> 39.2 mm
- net Net-(J6-Pin_1): track 39.7 -> 43.2 mm
- net Net-(J6-Pin_3): track 35.5 -> 38.7 mm
- net Net-(J6-Pin_4): track 31.4 -> 34.6 mm
- net Net-(D1-A): track 16.9 -> 16.0 mm
Other:
- board size 58.2 x 80.5 mm -> 56.6 x 77.5 mm
- board text added: "3.3V"
- board text added: "5V"
- board text added: "AGND"
- board text added: "AI0"
- board text added: "AI1"
- board text added: "AI2"
- board text added: "AI3"
- board text added: "AO0"
- board text added: "AO1"
- board text added: "DGND"
- board text added: "DIO0/PWM0"
- board text added: "DIO1/PWM1"
- board text added: "DIO10/PWM6"
- board text added: "DIO11/PWM7"
- board text added: "DIO12/PWM8"
- board text added: "DIO13/PWM9"
- board text added: "DIO14/I2C SCL"
- board text added: "DIO15/I2C SDA"
- board text added: "DIO2/PWM2"
- board text added: "DIO3/PWM3"
- board text added: "DIO4/SPI CS"
- board text added: "DIO5/SPI CLK"
- board text added: "DIO6/SPI MISO"
- board text added: "DIO7/SPI MOSI"
- board text added: "DIO8/PWM4"
- board text added: "DIO9/PWM5"
- board text added: "UART.RX"
- board text added: "UART.TX"

Commit message: rio module and added better silkscreening
Other:
- board text added: "(G)"
- board text added: "(Y)"
- board text added: "12V"
- board text added: "GND"
Changed lines of the file:
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@@
+		)
+	)
+	(gr_text "(G)"
+		(at 101.5 114.25 90)
+		(layer "F.SilkS")
+		(effects
+			(font
+				(size 1 1)
+				(thickness 0.15)
+			)
 		)
 	)
@@
 			)
 			(justify left bottom)
+		)
+	)
+	(gr_text "(Y)"
+		(at 101.5 117 90)
+		(layer "F.SilkS")
+		(effects
+			(font
+				(size 1 1)
+				(thickness 0.15)
+			)
 		)
 	)
@@
 			)
 			(justify left bottom)
+		)
+	)
+	(gr_text "GND\n"
+		(at 101 133.5 90)
+		(layer "F.SilkS")
+		(effects
+			(font
+				(size 1 1)
+				(thickness 0.15)
+			)
+		)
+	)
+	(gr_text "GND\n"
+		(at 101.75 123.75 90)
+		(layer "F.SilkS")
+		(effects
+			(font
+				(size 1 1)
+				(thickness 0.15)
+			)
 		)
 	)
@@
 		)
 	)
+	(gr_text "12V"
+		(at 101.75 120.5 90)
+		(layer "F.SilkS")
+		(effects
+			(font
+				(size 1 1)
+				(thickness 0.15)
+			)
+		)
+	)
+	(gr_text "12V"
+		(at 100.75 129.75 90)
+		(layer "F.SilkS")
+		(effects
+			(font
+				(size 1 1)
+				(thickness 0.15)
+			)
+		)
+	)

Commit message: added features claimed to be from previous commit
Parts:
- added J10: Conn_01x03_Pin, custom:Molex_SL_171971-0003_1x03_P2.54mm_Vertical, F.Cu at (106.2, 157.0)
- added J7: Conn_01x04_Pin, custom:Molex_SL_171971-0004_1x04_P2.54mm_Vertical, F.Cu at (115.0, 143.2)
- added J8: Conn_01x04_Pin, custom:Molex_SL_171971-0004_1x04_P2.54mm_Vertical, F.Cu at (106.2, 143.2)
- added J9: Conn_01x03_Pin, custom:Molex_SL_171971-0003_1x03_P2.54mm_Vertical, F.Cu at (115.0, 157.0)
- J5: value Conn_02x17_Odd_Even -> Conn_01x04_Pin; footprint Connector_PinSocket_2.54mm:PinSocket_2x17_P2.54mm_Vertical -> custom:Molex_SL_171971-0004_1x04_P2.54mm_Vertical
- J6: value Conn_01x04_Socket -> Conn_01x04_Pin; footprint Connector_PinSocket_2.54mm:PinSocket_1x04_P2.54mm_Vertical -> custom:Molex_SL_171971-0004_1x04_P2.54mm_Vertical
- moved J5 28.7 mm to (132.5, 143.2)
- moved J6 17.9 mm to (123.8, 143.2), turned to -90 degrees
- moved J2 0.78 mm to (107.5, 129.0)
Connections:
- J4 pad 5: Net-(J6-Pin_1) -> Net-(U1-MXP_DIO0_PWM0)
- J4 pad 6: Net-(J6-Pin_2) -> Net-(U1-MXP_DIO1_PWM1)
- J4 pad 7: Net-(J6-Pin_3) -> Net-(U1-MXP_DIO2_PWM2)
- J4 pad 8: Net-(J6-Pin_4) -> Net-(U1-MXP_DIO3_PWM3)
- J5 pad 1: Net-(J5-Pin_1) -> /12v
- J5 pad 4: Net-(J5-Pin_4) -> /GND
- J6 pad 1: Net-(J6-Pin_1) -> /12v
- J6 pad 4: Net-(J6-Pin_4) -> /GND
- U1 pad 1: Net-(J5-Pin_1) -> Net-(J10-Pin_2)
- U1 pad 10: Net-(J5-Pin_10) -> unconnected-(U1-MXP_RX-Pad10)
- U1 pad 11: Net-(J5-Pin_11) -> Net-(U1-MXP_DIO0_PWM0)
- U1 pad 12: /DGND -> /GND
- U1 pad 13: Net-(J5-Pin_13) -> Net-(U1-MXP_DIO1_PWM1)
- U1 pad 14: Net-(J5-Pin_14) -> unconnected-(U1-MXP_TX-Pad14)
- U1 pad 15: Net-(J5-Pin_15) -> Net-(U1-MXP_DIO2_PWM2)
- U1 pad 16: /DGND -> /GND
- U1 pad 17: Net-(J5-Pin_17) -> Net-(U1-MXP_DIO3_PWM3)
- U1 pad 18: Net-(J5-Pin_18) -> Net-(J10-Pin_1)
- U1 pad 19: Net-(J5-Pin_19) -> Net-(J5-Pin_2)
- U1 pad 2: Net-(J5-Pin_2) -> unconnected-(U1-MXP_AO0-Pad2)
- U1 pad 20: /DGND -> /GND
- U1 pad 21: Net-(J5-Pin_21) -> Net-(J5-Pin_3)
- U1 pad 22: Net-(J5-Pin_22) -> Net-(J8-Pin_2)
- U1 pad 23: Net-(J5-Pin_23) -> Net-(J6-Pin_2)
- U1 pad 24: /DGND -> /GND
- U1 pad 25: Net-(J5-Pin_25) -> Net-(J6-Pin_3)
- U1 pad 26: Net-(J5-Pin_26) -> Net-(J8-Pin_3)
- U1 pad 27: Net-(J5-Pin_27) -> Net-(J7-Pin_2)
- U1 pad 28: /DGND -> /GND
- U1 pad 29: Net-(J5-Pin_29) -> Net-(J7-Pin_3)
- U1 pad 3: Net-(J5-Pin_3) -> unconnected-(U1-MXP_AI0-Pad3)
- U1 pad 30: /DGND -> /GND
- U1 pad 31: Net-(J5-Pin_31) -> Net-(J9-Pin_1)
- U1 pad 32: Net-(J5-Pin_32) -> unconnected-(U1-MXP_DIO14_SCL-Pad32)
- U1 pad 33: Net-(J5-Pin_33) -> unconnected-(U1-MXP_3V3-Pad33)
- U1 pad 34: Net-(J5-Pin_34) -> unconnected-(U1-MXP_DIO15_SDA-Pad34)
- U1 pad 4: Net-(J5-Pin_4) -> unconnected-(U1-MXP_AO1-Pad4)
- U1 pad 5: Net-(J5-Pin_5) -> unconnected-(U1-MXP_AI1-Pad5)
- U1 pad 6: /AGND -> /GND
- U1 pad 7: Net-(J5-Pin_7) -> unconnected-(U1-MXP_AI2-Pad7)
- U1 pad 8: /DGND -> /GND
- U1 pad 9: Net-(J5-Pin_9) -> unconnected-(U1-MXP_AI3-Pad9)
Routing:
- net /DGND: track 95.9 -> 0.00 mm
- net Net-(J8-Pin_2): track 0.00 -> 56.9 mm
- net Net-(U1-MXP_DIO1_PWM1): track 0.00 -> 54.1 mm
- net Net-(J10-Pin_2): track 0.00 -> 47.4 mm
- net Net-(U1-MXP_DIO0_PWM0): track 0.00 -> 45.6 mm
- net Net-(U1-MXP_DIO2_PWM2): track 0.00 -> 44.8 mm
- net Net-(U1-MXP_DIO3_PWM3): track 0.00 -> 44.3 mm
- net Net-(J6-Pin_1): track 43.2 -> 0.00 mm
- net Net-(J10-Pin_1): track 0.00 -> 42.3 mm
- net /12v: track 62.9 -> 103.6 mm
- net Net-(J8-Pin_3): track 0.00 -> 34.7 mm
- net Net-(J6-Pin_4): track 34.6 -> 0.00 mm
- net Net-(J7-Pin_2): track 0.00 -> 29.1 mm
- net Net-(J7-Pin_3): track 0.00 -> 25.9 mm
- net Net-(J5-Pin_2): track 8.89 -> 30.4 mm
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- removed copper zone on B.Cu, net /DGND
- removed copper zone on F.Cu, net /DGND
Other:
- board text added: "DIO 12 DIO 13"
- board text added: "DIO 4 DIO 5"
- board text added: "DIO 6 DIO 7"
- board text added: "DIO 8 DIO 9"
- board text added: "GND 2 1 12V"
- board text added: "GND 5V S"
- board text added: "PWM 6"
- board text added: "PWM 7"
- board text removed: "3.3V"
- board text removed: "5V"
- board text removed: "AGND"
- board text removed: "AI0"
- board text removed: "AI1"
- board text removed: "AI2"
- board text removed: "AI3"
- board text removed: "AO0"
- board text removed: "AO1"
- board text removed: "DGND"
- board text removed: "DIO0/PWM0"
- board text removed: "DIO1/PWM1"
- board text removed: "DIO10/PWM6"
- board text removed: "DIO11/PWM7"
- board text removed: "DIO12/PWM8"
- board text removed: "DIO13/PWM9"
- board text removed: "DIO14/I2C SCL"
- board text removed: "DIO15/I2C SDA"
- board text removed: "DIO2/PWM2"
- board text removed: "DIO3/PWM3"
- board text removed: "DIO4/SPI CS"
- board text removed: "DIO5/SPI CLK"
- board text removed: "DIO6/SPI MISO"
- board text removed: "DIO7/SPI MOSI"
- board text removed: "DIO8/PWM4"
- board text removed: "DIO9/PWM5"
- board text removed: "UART.RX"
- board text removed: "UART.TX"

Commit message: in a rush, changes made
Routing:
- net /12v: track 103.6 -> 104.3 mm
Changed lines of the file:
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@@
 		)
 		(model "/home/ben/Documents/CAN-over-RJ45/libs/2162711030.stp"
+			(hide yes)
 			(offset
 				(xyz -1.7 1.25 17)
@@
 		)
 		(model "/home/ben/Documents/CAN-over-RJ45/libs/2162711040.stp"
+			(hide yes)
 			(offset
 				(xyz -0.5 1.5 18)
@@
 		)
 		(model "/home/ben/Documents/CAN-over-RJ45/libs/2162711040.stp"
+			(hide yes)
 			(offset
 				(xyz -0.5 1.5 18)
@@
 		)
 		(model "/home/ben/Documents/CAN-over-RJ45/libs/2162711040.stp"
+			(hide yes)
 			(offset
 				(xyz -0.5 1.5 18)
@@
 		)
 		(model "/home/ben/Documents/CAN-over-RJ45/libs/2162711030.stp"
+			(hide yes)
 			(offset
 				(xyz -1.7 1.25 17)
@@
 		)
 		(model "/home/ben/Documents/CAN-over-RJ45/libs/2162711040.stp"
+			(hide yes)
 			(offset
 				(xyz -0.5 1.5 18)
@@
 	)
 	(segment
+		(start 149.320549 135.441)
+		(end 150.085 134.676549)
+		(width 0.8)
+		(layer "B.Cu")
+		(net 4)
+	)
+	(segment
 		(start 132.5 143.17)
 		(end 123.75 143.17)
-		(width 0.4)
+		(width 0.8)
 		(layer "B.Cu")
 		(net 4)
 	)
 	(segment
-		(start 144.925 136.261)
-		(end 148.217706 136.261)
-		(width 0.4)
+		(start 133.4 129.086)
+		(end 125.125 120.811)
+		(width 0.8)
 		(layer "B.Cu")
 		(net 4)
 	)
 	(segment
-		(start 137.75 129.086)
-		(end 144.925 136.261)
-		(width 0.4)
+		(start 148.25 136.5)
+		(end 149.309 135.441)
+		(width 0.8)
 		(layer "B.Cu")
 		(net 4)
 	)
 	(segment
-		(start 133.4 129.086)
-		(end 125.125 120.811)
-		(width 0.4)
+		(start 145.164 136.5)
+		(end 148.25 136.5)
+		(width 0.8)
 		(layer "B.Cu")
 		(net 4)
@@
 		(start 133.4 142.27)
 		(end 132.5 143.17)
-		(width 0.4)
+		(width 0.8)
 		(layer "B.Cu")
 		(net 4)
@@
 		(start 123.75 143.17)
 		(end 115 143.17)
-		(width 0.4)
+		(width 0.8)
 		(layer "B.Cu")
 		(net 4)
 	)
 	(segment
-		(start 149.885 134.593706)
-		(end 149.885 131.161)
-		(width 0.4)
+		(start 133.4 129.086)
+		(end 133.4 142.27)
+		(width 0.8)
 		(layer "B.Cu")
 		(net 4)
 	)
 	(segment
-		(start 133.4 129.086)
-		(end 133.4 142.27)
-		(width 0.4)
+		(start 149.309 135.441)
+		(end 149.320549 135.441)
+		(width 0.8)
 		(layer "B.Cu")
 		(net 4)
@@
 	(segment
 		(start 137.75 129.086)
-		(end 140.11 129.086)
-		(width 0.4)
+		(end 145.164 136.5)
+		(width 0.8)
 		(layer "B.Cu")
 		(net 4)
 	)
 	(segment
-		(start 149.885 131.161)
-		(end 148.78 130.056)
-		(width 0.4)
+		(start 137.75 129.086)
+		(end 140.11 129.086)
+		(width 0.8)
 		(layer "B.Cu")
 		(net 4)
@@
 		(start 140.11 129.086)
 		(end 142.18 127.016)
-		(width 0.4)
+		(width 0.8)
 		(layer "B.Cu")
 		(net 4)
@@
 		(start 133.4 129.086)
 		(end 137.75 129.086)
-		(width 0.4)
+		(width 0.8)
+		(layer "B.Cu")
+		(net 4)
+	)
+	(segment
+		(start 150.085 134.665)
+		(end 150.25 134.5)
+		(width 0.8)
 		(layer "B.Cu")
 		(net 4)
@@
 		(start 115 143.17)
 		(end 106.25 143.17)
-		(width 0.4)
+		(width 0.8)
 		(layer "B.Cu")
 		(net 4)
 	)
 	(segment
-		(start 148.217706 136.261)
-		(end 149.885 134.593706)
-		(width 0.4)
+		(start 150.25 134.5)
+		(end 150.25 131.526)
+		(width 0.8)
 		(layer "B.Cu")
 		(net 4)
@@
 		(start 125.125 120.811)
 		(end 104.32 120.811)
-		(width 0.4)
+		(width 0.8)
+		(layer "B.Cu")
+		(net 4)
+	)
+	(segment
+		(start 150.085 134.676549)
+		(end 150.085 134.665)
+		(width 0.8)
+		(layer "B.Cu")
+		(net 4)
+	)
+	(segment
+		(start 150.25 131.526)
+		(end 148.78 130.056)
+		(width 0.8)
 		(layer "B.Cu")
 		(net 4)
@@
 		(start 107.5 129)
 		(end 112.5 129)
-		(width 0.4)
+		(width 0.8)
 		(layer "B.Cu")
 		(net 8)
@@
 		(start 112.5 129)
 		(end 123.154 129)
-		(width 0.4)
+		(width 0.8)
 		(layer "B.Cu")
 		(net 8)

Commit message: final major changes, exported for JLCPCB
Parts:
- added REF**: PinSocket_1x04_P2.54mm_Horizontal, Connector_PinSocket_2.54mm:PinSocket_1x04_P2.54mm_Horizontal, F.Cu at (101.8, 118.3)
- moved J1 7.41 mm to (104.2, 121.7)
- moved J3 5.26 mm to (109.5, 121.7)
- moved D1 4.74 mm to (128.7, 129.0)
Connections:
- D1 pad 1: /12v -> 12Vu
Routing:
- net 12Vu: track 0.00 -> 35.3 mm
- net /12v: track 104.3 -> 112.9 mm
- net Net-(D1-A): track 15.8 -> 11.0 mm
- net Net-(J1-Pin_1): track 50.1 -> 48.5 mm
- net Net-(J1-Pin_2): track 49.0 -> 49.6 mm
Other:
- outline, holes or cut-outs redrawn
